File: hardware/IAuto.kicad_pcb (KiCad board)
At the start: 2 copper layers, 56 x 85 mm, 66 parts, among them J1 Barrel_Jack_Switch, J2 4R7uH, J3 4R7uH, J4 M1, J5 M2, J6 Cable_PAD, J7 Cable_PAD, J8 Cable_PAD, J9 Cable_PAD, P1 CONN_02X20, P2 CONN_02X05, Q1 SI4835DDY-T1-GE3, Q2 2N7002, Q3 2N7002, Q4 2N7002, Q5 2N7002, U1 ESP32_NODEMCU, U2 MP1584, U3 MP1584, U4 DRV8833

Commit message: Hardware
Routing:
- net /Logical Part/GPIO26: track 79.9 -> 79.3 mm

Commit message: anteultimos_cambios
Parts:
- removed Q2, Q4: 2N7002, EESTN5:SOT23
- removed R16, R18, R20, R22: 10K, EESTN5:R_0805
- P2: value CONN_02X05 -> CONN_02x6; footprint MacroLib:Pin_strip_02x05 -> MacroLib:Pin_strip_2x6
- moved P2 1.40 mm to (170.8, 78.2), turned to 90 degrees
Connections:
- J4 pad 1: /Power Part/BOUT1 -> /Power Part/A1
- J4 pad 2: GND -> (no net)
- J4 pad 3: /Power Part/B1 -> +5V
- J4 pad 4: /Power Part/A1 -> GND
- J4 pad 5: +5V -> /Power Part/BOUT1
- J5 pad 1: Net-(F4-Pad2) -> /Power Part/A2
- J5 pad 2: +5V -> (no net)
- J5 pad 3: /Power Part/A2 -> GND
- J5 pad 4: /Power Part/B2 -> +5V
- J5 pad 5: GND -> /Power Part/AOUT1
- J5 pad 6: /Power Part/AOUT1 -> Net-(F4-Pad2)
- P2 pad 10: +5VF -> /Logical Part/F+3.3V
- P2 pad 6: /Logical Part/GPIO23 -> /Logical Part/GPIO18
- P2 pad 8: /Logical Part/F+3.3V -> /Logical Part/GPIO19
- P2 pad 9: GND -> /Logical Part/GPIO34
- R1 pad 2: GPIO34 -> GPIO39
- R2 pad 1: GPIO34 -> GPIO39
- U1 pad 30: AIN2 -> /Logical Part/GPIO18
- U1 pad 31: AIN1 -> /Logical Part/GPIO19
- U1 pad 33: BO2 -> AIN2
- U1 pad 36: AO2 -> AIN1
- U1 pad 37: /Logical Part/GPIO23 -> AO2
- U1 pad 4: BO1 -> AO1
- U1 pad 5: AO1 -> GPIO39
- U1 pad 6: GPIO34 -> /Logical Part/GPIO34
Routing:
- net /Logical Part/GPIO34: track 0.00 -> 110.3 mm, vias 0 -> 1
- net +5V: track 204.5 -> 109.0 mm, vias 5 -> 2
- net GPIO39: track 0.00 -> 83.8 mm, vias 0 -> 1
- net GPIO34: track 79.2 -> 0.00 mm, vias 2 -> 0
- net /Power Part/BOUT1: track 47.9 -> 0.00 mm, vias 1 -> 0
- net /Logical Part/GPIO23: track 37.8 -> 0.00 mm
- net +3V3: track 110.0 -> 78.3 mm
- net /Power Part/A2: track 30.7 -> 2.58 mm
- net /Power Part/A1: track 30.7 -> 2.67 mm
- net /Power Part/B2: track 27.1 -> 0.00 mm
- net /Power Part/B1: track 26.5 -> 0.00 mm
- net /Logical Part/GPIO19: track 0.00 -> 21.9 mm
- net /Logical Part/GPIO18: track 0.00 -> 20.8 mm
- net BO1: track 13.1 -> 0.00 mm
- net AO1: track 20.5 -> 33.6 mm
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Other:
- net class Default: clearance 0.127 -> 0.2032; via_dia 0.5 -> 0.508; via_drill 0.3 -> 0.3048
- rule trace_clearance: 0.127 -> 0.2032
- rule trace_min: 0.2 -> 0.254
- rule via_min_drill: 0.3 -> 0.254
- rule via_min_size: 0.4 -> 0.4064

Commit message: ultimos cambios
Parts:
- added J10: Cable_PAD, EESTN5:LOGO_EESTN5, B.Cu at (150.2, 112.2)
- U1: footprint MacroLib:NodeMCU-ESP32 -> IAuto:NodeMCU-ESP32
- moved F1 19.7 mm to (153.7, 52.7), turned to 0 degrees
- moved F4 14.8 mm to (154.7, 60.2)
- moved Q5 8.41 mm to (154.2, 47.0)
- moved R21 8.41 mm to (154.2, 49.9)
- moved R23 8.41 mm to (154.2, 44.1)
- moved R19 7.86 mm to (142.2, 58.6), turned to 180 degrees
- moved R17 5.80 mm to (142.2, 52.8), turned to 180 degrees
- moved F3 4.93 mm to (147.2, 49.9)
- moved Q3 3.69 mm to (142.2, 55.7), turned to 180 degrees
- moved R29 1.18 mm to (153.9, 74.8)
- moved J2 0.92 mm to (139.6, 105.2)
- moved C7 0.73 mm to (133.8, 105.6)
- moved U3 0.48 mm to (145.4, 91.0)
- moved R8 0.31 mm to (143.8, 96.4)
- moved R24 0.13 mm to (144.1, 67.4)
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Connections:
- F4 pad 1: /Power Part/AOUT2 -> /Power Part/AOUT1
- J5 pad 5: /Power Part/AOUT1 -> /Power Part/AOUT2
Routing:
- net +5V: track 109.0 -> 188.6 mm, vias 2 -> 1
- net +3V3: track 78.3 -> 29.3 mm, vias 4 -> 0
- net /Power Part/AOUT1: track 49.3 -> 6.48 mm, vias 1 -> 0
- net /Power Part/BOUT1: track 0.00 -> 37.6 mm, vias 0 -> 1
- net /Logical Part/F+3.3V: track 7.72 -> 33.7 mm, vias 0 -> 1
- net AO1: track 33.6 -> 8.94 mm
- net /Power Part/A1: track 2.67 -> 22.9 mm
- net /Power Part/A2: track 2.58 -> 16.4 mm
- net AIN1: track 21.7 -> 33.0 mm
- net AO2: track 20.7 -> 10.1 mm
- net GND: track 10.7 -> 18.8 mm
- net /Power Part/AOUT2: track 20.1 -> 27.1 mm
- net /Power Part/BOUT2: track 19.2 -> 12.5 mm
- net Net-(F4-Pad2): track 18.6 -> 14.8 mm
- net AIN2: track 33.7 -> 31.0 mm
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
Commit message: Final
Parts:
- removed J10: Cable_PAD, EESTN5:LOGO_EESTN5
- added G***: LOGO, EESTN5:Logo_silk_OSHW_12x13mm, B.Cu at (148.3, 68.8)
- added G***: LOGO, EESTN5:LOGO_EESTN5, B.Cu at (148.3, 95.8)
- added REF***: KiCad-Logo2_8mm_SilkScreen, EESTN5:KiCad-Logo2_8mm_SilkScreen, B.Cu at (148.2, 82.8)
- J4, J5: footprint MacroLib:JST_XH_1X6 -> IAuto:Conector_jst_6_pins_2mm
- moved J4 0.99 mm to (130.7, 48.3), turned to 270 degrees
- moved J5 0.97 mm to (168.3, 48.3), turned to 90 degrees
Connections:
- J4 pad 1: /Power Part/A1 -> Net-(F3-Pad2)
- J4 pad 2: (no net) -> /Power Part/BOUT1
- J4 pad 3: +5V -> GND
- J4 pad 4: GND -> +5V
- J4 pad 5: /Power Part/BOUT1 -> (no net)
- J4 pad 6: Net-(F3-Pad2) -> /Power Part/A1
- J5 pad 1: /Power Part/A2 -> Net-(F4-Pad2)
- J5 pad 2: (no net) -> /Power Part/AOUT2
- J5 pad 3: GND -> +5V
- J5 pad 4: +5V -> GND
- J5 pad 5: /Power Part/AOUT2 -> (no net)
- J5 pad 6: Net-(F4-Pad2) -> /Power Part/A2
Routing:
- net /Power Part/BOUT1: track 37.6 -> 39.9 mm
- net /Power Part/A2: track 16.4 -> 18.4 mm
- net Net-(F3-Pad2): track 19.1 -> 20.6 mm
- net Net-(F4-Pad2): track 14.8 -> 16.3 mm
- net /Power Part/AOUT2: track 27.1 -> 28.4 mm
- net +5V: track 188.6 -> 189.6 mm

Commit message: hardware_v20
Parts:
- removed REF***: KiCad-Logo2_8mm_SilkScreen, EESTN5:KiCad-Logo2_8mm_SilkScreen
- added C12: 1000uF/16V, EESTN5:CAP_ELEC_8x11.5mm, F.Cu at (132.8, 113.6)
- added R16: 47k, EESTN5:R_0805, F.Cu at (152.3, 61.6)
- U4: footprint MacroLib:HTSSOP -> MacroLib:HTSSOPP
- moved G*** 16.6 mm to (148.5, 79.1)
- moved G*** 14.6 mm to (148.5, 54.2)
- moved C9 9.98 mm to (148.1, 76.0), turned to 0 degrees
- moved C11 8.32 mm to (153.5, 67.1)
- moved F4 3.28 mm to (152.2, 58.1), turned to 0 degrees
- moved C7 1.80 mm to (133.8, 103.8)
- moved C10 1.46 mm to (148.3, 73.4), turned to 0 degrees
- moved R14 1.08 mm to (142.3, 80.0), turned to 90 degrees
- turned C8 to 0 degrees
Connections:
- U4 pad 1: /Power Part/VM -> Net-(R16-Pad2)
Routing:
- net +5V: track 189.6 -> 201.1 mm
- net GND: track 18.8 -> 7.71 mm, vias 46 -> 50
- net /Power Part/VM: track 42.2 -> 46.3 mm
- net Net-(R16-Pad2): track 0.00 -> 3.46 mm
- net Net-(C11-Pad2): track 3.58 -> 7.01 mm
- net Net-(R25-Pad1): track 6.84 -> 9.51 mm
- net /Power Part/AOUT2: track 28.4 -> 30.9 mm
- net Net-(F4-Pad2): track 16.3 -> 17.3 mm
- net Net-(C4-Pad1): track 3.68 -> 3.09 mm
- net /Power Part/BOUT1: track 39.9 -> 39.4 mm
