File: hardware/Loguica.sch (KiCad schematic (older format))
At the start: 8 parts, among them P1 CONN_02X20, P2 CONN_02X05, U1 ESP32_NODEMCU

Commit message: hardware
Connections:
- net AIN2: now also U1.9 (GPIO33); no longer U1.29 (GPIO5)
- net CS: now also U1.8 (GPIO32); no longer U1.23 (GPIO15)
- net GPIO32: no longer U1.8 (GPIO32)
- net GPIO33 renamed GPIO5
- net GPIO5: now also U1.29 (GPIO5); no longer U1.9 (GPIO33)
- new net GPIO15: U1.23 (GPIO15)
Changed lines of the file:
@@
 Text Label 2750 3700 2    50   ~ 0
 CLK
-Text Label 4750 4100 0    50   ~ 0
-CS
 Text GLabel 4500 3300 2    50   Input ~ 0
 AIN1
-Text GLabel 4500 3500 2    50   Input ~ 0
+Text GLabel 3000 3300 0    50   Input ~ 0
 AIN2
 Text GLabel 4500 3400 2    50   Input ~ 0
@@
 	4500 3400 4400 3400
 Wire Wire Line
-	4500 3500 4400 3500
+	4750 3500 4400 3500
 Text GLabel 3000 2900 0    50   Input ~ 0
 AO1
@@
 	3100 3200 2650 3200
 Wire Wire Line
-	3100 3300 2650 3300
+	3100 3300 3000 3300
 Wire Wire Line
 	3100 3400 2650 3400
 Wire Wire Line
 	3100 3500 2650 3500
-Text Label 2650 3200 2    50   ~ 0
-GPIO32
-Text Label 2650 3300 2    50   ~ 0
-GPIO33
+Text Label 4750 4100 0    50   ~ 0
+GPIO15
+Text Label 4750 3500 0    50   ~ 0
+GPIO5
 Text Label 2650 3400 2    50   ~ 0
 GPIO25
@@
 Wire Wire Line
 	4500 2700 4400 2700
-Text GLabel 7350 3450 2    50   Input ~ 0
+Text GLabel 7100 3450 2    50   Input ~ 0
 +5VF
 $Comp
@@
 GPIO32
 Text Label 7100 3150 0    50   ~ 0
-GPIO33
+GPIO5
 Text Label 7100 3350 0    50   ~ 0
 GPIO26
@@
 	7100 3550 7000 3550
 Wire Wire Line
-	7350 3450 7000 3450
+	7100 3450 7000 3450
 Text Label 2300 2600 2    50   ~ 0
 F+3.3V
@@
 Wire Wire Line
 	4150 5700 4150 5950
+Text Label 2650 3200 2    50   ~ 0
+CS
 $EndSCHEMATC

Commit message: hardware
Connections:
- net GPIO15 is gone; now on net CS: U1.23 (GPIO15)
- net +5VF: now also P2.10 (P10); no longer P2.8 (P8)
- net AIN2: now also U1.30 (GPIO18); no longer U1.9 (GPIO33)
- net AO2: now also U1.36 (GPIO22); no longer U1.24 (GPIO2)
- net BIN1: now also U1.9 (GPIO33); no longer U1.30 (GPIO18)
- net BO2: now also U1.33 (GPIO21); no longer U1.26 (GPIO4)
- net CLK: now also U1.16 (GPIO13); no longer U1.13 (GPIO14)
- net CS: no longer U1.8 (GPIO32)
- net F+3.3V: now also P2.8 (P8); no longer P2.7 (P7)
- net GND: no longer P2.10 (P10)
- net GPIO0: now also P2.2 (P2); no longer P2.5 (P5)
- net GPIO23: now also P2.6 (P6)
- net GPIO25: now also P2.1 (P1); no longer P2.3 (P3)
- net GPIO26: now also P2.3 (P3); no longer P2.6 (P6)
- net GPIO32: now also P2.5 (P5), U1.8 (GPIO32); no longer P2.4 (P4)
- net GPIO34: now also U1.6 (GPIO34); no longer P2.1 (P1), U1.7 (GPIO35)
- net GPIO35: now also P2.7 (P7), U1.7 (GPIO35); no longer U1.6 (GPIO34)
- net GPIO5: now also P2.4 (P4); no longer P2.2 (P2)
- net MOSI: now also U1.13 (GPIO14); no longer U1.16 (GPIO13)
- net RXD: now also U1.24 (GPIO2); no longer U1.27 (GPIO16)
- net SCL: now also U1.27 (GPIO16); no longer U1.36 (GPIO22)
- net SDA: now also U1.28 (GPIO17); no longer U1.33 (GPIO21)
- net TXD: now also U1.26 (GPIO4); no longer U1.28 (GPIO17)
- net +3V3: now reaches F1.2, U1.2 (3V3)
Other:
- moved on the sheet: F1, R26, R27, R28, R29
Changed lines of the file:
@@
 Wire Wire Line
 	4750 3900 4400 3900
-Text Label 4750 3700 0    50   ~ 0
+Text Label 4500 4000 0    50   ~ 0
 RXD
-Text Label 4750 3600 0    50   ~ 0
+Text Label 4500 3800 0    50   ~ 0
 TXD
 $Comp
@@
 Wire Wire Line
 	8750 3600 8650 3600
-Text Label 3000 4000 2    50   ~ 0
+Text Label 2750 3700 2    50   ~ 0
 MOSI
 Text Label 2750 3800 2    50   ~ 0
 MISO
-Text Label 2750 3700 2    50   ~ 0
+Text Label 3000 4000 2    50   ~ 0
 CLK
 Text GLabel 4500 3300 2    50   Input ~ 0
 AIN1
+Text GLabel 4500 3400 2    50   Input ~ 0
+AIN2
 Text GLabel 3000 3300 0    50   Input ~ 0
-AIN2
-Text GLabel 4500 3400 2    50   Input ~ 0
 BIN1
 Text GLabel 3000 3600 0    50   Input ~ 0
@@
 Text GLabel 3000 2800 0    50   Input ~ 0
 BO1
-Text GLabel 4500 4000 2    50   Input ~ 0
+Text GLabel 4500 2800 2    50   Input ~ 0
 AO2
-Text GLabel 4500 3800 2    50   Input ~ 0
+Text GLabel 4500 3100 2    50   Input ~ 0
 BO2
 Wire Wire Line
@@
 	4500 3800 4400 3800
 Text Label 2650 3100 2    50   ~ 0
-GPIO34
+GPIO35
 Wire Wire Line
 	3000 3000 3100 3000
@@
 Wire Wire Line
 	3100 3500 2650 3500
-Text Label 4750 4100 0    50   ~ 0
-GPIO15
+Text Label 2650 3200 2    50   ~ 0
+GPIO32
 Text Label 4750 3500 0    50   ~ 0
 GPIO5
@@
 Text Label 2650 3500 2    50   ~ 0
 GPIO26
-Text Label 4500 2700 0    50   ~ 0
-GPIO23
-Wire Wire Line
-	4500 2700 4400 2700
-Text GLabel 7100 3450 2    50   Input ~ 0
+Text GLabel 7100 3550 2    50   Input ~ 0
 +5VF
 $Comp
@@
 	1    0    0    -1
 $EndComp
-Text Label 4500 3100 0    50   ~ 0
+Text Label 4750 3600 0    50   ~ 0
 SDA
-Text Label 4500 2800 0    50   ~ 0
+Text Label 4750 3700 0    50   ~ 0
 SCL
 Wire Wire Line
+	4500 3100 4400 3100
+Wire Wire Line
 	4500 2800 4400 2800
-Wire Wire Line
-	4500 3100 4400 3100
 Wire Wire Line
 	3000 4000 3100 4000
@@
 Wire Wire Line
 	3000 4400 3100 4400
-Text Label 6400 3150 2    50   ~ 0
-GPIO34
+Text Label 6400 3450 2    50   ~ 0
+GPIO35
+Text Label 6400 3350 2    50   ~ 0
+GPIO32
 Text Label 7100 3250 0    50   ~ 0
-GPIO32
-Text Label 7100 3150 0    50   ~ 0
 GPIO5
-Text Label 7100 3350 0    50   ~ 0
+Text Label 6400 3250 2    50   ~ 0
 GPIO26
 $Comp
@@
 	6400 3250 6500 3250
 Wire Wire Line
-	6400 3450 6500 3450
+	7100 3550 7000 3550
 Wire Wire Line
 	7100 3150 7000 3150
@@
 L power:GND #PWR06
 U 1 1 60E92CD9
-P 7100 3750
-F 0 "#PWR06" H 7100 3500 50  0001 C CNN
-F 1 "GND" H 7105 3577 50  0000 C CNN
-F 2 "" H 7100 3750 50  0001 C CNN
-F 3 "" H 7100 3750 50  0001 C CNN
-	1    7100 3750
-	1    0    0    -1
-$EndComp
-Wire Wire Line
-	7100 3750 7100 3650
-Wire Wire Line
-	7100 3550 7000 3550
+P 6400 3750
+F 0 "#PWR06" H 6400 3500 50  0001 C CNN
+F 1 "GND" H 6405 3577 50  0000 C CNN
+F 2 "" H 6400 3750 50  0001 C CNN
+F 3 "" H 6400 3750 50  0001 C CNN
+	1    6400 3750
+	-1   0    0    -1
+$EndComp
+Wire Wire Line
+	6400 3550 6500 3550
 Wire Wire Line
 	7100 3450 7000 3450
-Text Label 2300 2600 2    50   ~ 0
+Text Label 2150 2600 2    50   ~ 0
 F+3.3V
-$Comp
-L MacroLib:FUSE F1
-U 1 1 60E10EEE
-P 2700 2600
-F 0 "F1" H 2700 2825 50  0000 C CNN
-F 1 "FUSE 0,5A" H 2700 2734 50  0000 C CNN
-F 2 "EESTN5:R_1206" H 2700 2700 50  0001 C CNN
-F 3 "" H 2700 2700 50  0001 C CNN
-	1    2700 2600
-	1    0    0    -1
-$EndComp
-Wire Wire Line
-	2300 2600 2400 2600
-Wire Wire Line
-	3000 2600 3100 2600
-Wire Wire Line
-	6400 3550 6500 3550
-Text Label 6400 3450 2    50   ~ 0
+Wire Wire Line
+	2150 2600 2250 2600
+Text Label 7100 3450 0    50   ~ 0
 F+3.3V
 Wire Wire Line
 	6400 3350 6500 3350
-Text Label 6400 3350 2    50   ~ 0
+Text Label 7100 3150 0    50   ~ 0
 GPIO0
-Text Label 6400 3250 2    50   ~ 0
+Text Label 6400 3150 2    50   ~ 0
 GPIO25
-Wire Wire Line
-	6400 3550 6400 3650
-Wire Wire Line
-	6400 3650 7100 3650
-Connection ~ 7100 3650
-Wire Wire Line
-	7100 3650 7100 3550
 Text GLabel 3000 3000 0    50   Input ~ 0
-GPIO35
+GPIO34
 Wire Notes Line
 	8050 1800 8050 5000
@@
 	5750 1800 7900 1800
 Wire Notes Line
-	5600 5000 1700 5000
-Wire Notes Line
-	1700 5000 1700 1800
-Wire Notes Line
-	5600 5000 5600 1800
+	5600 6200 1700 6200
+Wire Notes Line
+	1700 6200 1700 1800
+Wire Notes Line
+	5600 6200 5600 1800
 Wire Notes Line
 	5600 1800 1700 1800
@@
 	1    0    0    -1
 $EndComp
-Text GLabel 4750 5700 2    50   Input ~ 0
+Text GLabel 3850 5100 2    50   Input ~ 0
 AIN1
-Text GLabel 4750 6200 2    50   Input ~ 0
+Text GLabel 3850 5600 2    50   Input ~ 0
 AIN2
-Text GLabel 4750 5950 2    50   Input ~ 0
+Text GLabel 3850 5350 2    50   Input ~ 0
 BIN1
-Text GLabel 4750 5450 2    50   Input ~ 0
+Text GLabel 3850 4850 2    50   Input ~ 0
 BIN2
 $Comp
 L EESTN5:R R26
 U 1 1 61313539
-P 4450 5450
-F 0 "R26" V 4265 5450 50  0000 C CNN
-F 1 "R" V 4356 5450 50  0000 C CNN
-F 2 "EESTN5:R_0805" H 4450 5450 60  0001 C CNN
-F 3 "" H 4450 5450 60  0000 C CNN
-	1    4450 5450
+P 3550 4850
+F 0 "R26" V 3365 4850 50  0000 C CNN
+F 1 "R" V 3456 4850 50  0000 C CNN
+F 2 "EESTN5:R_0805" H 3550 4850 60  0001 C CNN
+F 3 "" H 3550 4850 60  0000 C CNN
+	1    3550 4850
 	0    1    1    0
 $EndComp
@@
 L EESTN5:R R27
 U 1 1 61313917
-P 4450 5700
-F 0 "R27" V 4265 5700 50  0000 C CNN
-F 1 "R" V 4356 5700 50  0000 C CNN
-F 2 "EESTN5:R_0805" H 4450 5700 60  0001 C CNN
-F 3 "" H 4450 5700 60  0000 C CNN
-	1    4450 5700
+P 3550 5100
+F 0 "R27" V 3365 5100 50  0000 C CNN
+F 1 "R" V 3456 5100 50  0000 C CNN
+F 2 "EESTN5:R_0805" H 3550 5100 60  0001 C CNN
+F 3 "" H 3550 5100 60  0000 C CNN
+	1    3550 5100
 	0    1    1    0
 $EndComp
@@
 L EESTN5:R R28
 U 1 1 61313A99
-P 4450 5950
-F 0 "R28" V 4265 5950 50  0000 C CNN
-F 1 "R" V 4356 5950 50  0000 C CNN
-F 2 "EESTN5:R_0805" H 4450 5950 60  0001 C CNN
-F 3 "" H 4450 5950 60  0000 C CNN
-	1    4450 5950
+P 3550 5350
+F 0 "R28" V 3365 5350 50  0000 C CNN
+F 1 "R" V 3456 5350 50  0000 C CNN
+F 2 "EESTN5:R_0805" H 3550 5350 60  0001 C CNN
+F 3 "" H 3550 5350 60  0000 C CNN
+	1    3550 5350
 	0    1    1    0
 $EndComp
@@
 L EESTN5:R R29
 U 1 1 61313D18
-P 4450 6200
-F 0 "R29" V 4265 6200 50  0000 C CNN
-F 1 "R" V 4356 6200 50  0000 C CNN
-F 2 "EESTN5:R_0805" H 4450 6200 60  0001 C CNN
-F 3 "" H 4450 6200 60  0000 C CNN
-	1    4450 6200
+P 3550 5600
+F 0 "R29" V 3365 5600 50  0000 C CNN
+F 1 "R" V 3456 5600 50  0000 C CNN
+F 2 "EESTN5:R_0805" H 3550 5600 60  0001 C CNN
+F 3 "" H 3550 5600 60  0000 C CNN
+	1    3550 5600
 	0    1    1    0
 $EndComp
@@
 L power:GND #PWR031
 U 1 1 6132838D
-P 4150 6400
-F 0 "#PWR031" H 4150 6150 50  0001 C CNN
-F 1 "GND" H 4155 6227 50  0000 C CNN
-F 2 "" H 4150 6400 50  0001 C CNN
-F 3 "" H 4150 6400 50  0001 C CNN
-	1    4150 6400
-	1    0    0    -1
-$EndComp
-Wire Wire Line
-	4150 6400 4150 6200
-Wire Wire Line
-	4150 6200 4350 6200
-Wire Wire Line
-	4350 5950 4150 5950
-Wire Wire Line
-	4150 5950 4150 6200
-Connection ~ 4150 6200
-Wire Wire Line
-	4550 6200 4750 6200
-Wire Wire Line
-	4550 5950 4750 5950
-Wire Wire Line
-	4550 5700 4750 5700
-Wire Wire Line
-	4550 5450 4750 5450
-Wire Wire Line
-	4350 5450 4150 5450
-Wire Wire Line
-	4150 5450 4150 5700
-Connection ~ 4150 5950
-Wire Wire Line
-	4350 5700 4150 5700
-Connection ~ 4150 5700
-Wire Wire Line
-	4150 5700 4150 5950
-Text Label 2650 3200 2    50   ~ 0
+P 3250 5800
+F 0 "#PWR031" H 3250 5550 50  0001 C CNN
+F 1 "GND" H 3255 5627 50  0000 C CNN
+F 2 "" H 3250 5800 50  0001 C CNN
+F 3 "" H 3250 5800 50  0001 C CNN
+	1    3250 5800
+	1    0    0    -1
+$EndComp
+Wire Wire Line
+	3250 5800 3250 5600
+Wire Wire Line
+	3250 5600 3450 5600
+Wire Wire Line
+	3450 5350 3250 5350
+Wire Wire Line
+	3250 5350 3250 5600
+Connection ~ 3250 5600
+Wire Wire Line
+	3650 5600 3850 5600
+Wire Wire Line
+	3650 5350 3850 5350
+Wire Wire Line
+	3650 5100 3850 5100
+Wire Wire Line
+	3650 4850 3850 4850
+Wire Wire Line
+	3450 4850 3250 4850
+Wire Wire Line
+	3250 4850 3250 5100
+Connection ~ 3250 5350
+Wire Wire Line
+	3450 5100 3250 5100
+Connection ~ 3250 5100
+Wire Wire Line
+	3250 5100 3250 5350
+Text Label 4750 4100 0    50   ~ 0
 CS
+$Comp
+L MacroLib:FUSE F1
+U 1 1 60E10EEE
+P 2550 2600
+F 0 "F1" H 2550 2825 50  0000 C CNN
+F 1 "FUSE 0,5A" H 2550 2734 50  0000 C CNN
+F 2 "EESTN5:R_1206" H 2550 2700 50  0001 C CNN
+F 3 "" H 2550 2700 50  0001 C CNN
+	1    2550 2600
+	1    0    0    -1
+$EndComp
+Wire Wire Line
+	2850 2600 3000 2600
+$Comp
+L power:+3.3V #PWR0101
+U 1 1 61468625
+P 3000 2450
+F 0 "#PWR0101" H 3000 2300 50  0001 C CNN
+F 1 "+3.3V" H 3015 2623 50  0000 C CNN
+F 2 "" H 3000 2450 50  0001 C CNN
+F 3 "" H 3000 2450 50  0001 C CNN
+	1    3000 2450
+	1    0    0    -1
+$EndComp
+Wire Wire Line
+	3000 2450 3000 2600
+Connection ~ 3000 2600
+Wire Wire Line
+	3000 2600 3100 2600
+Wire Wire Line
+	4500 2700 4400 2700
+Text Label 4500 2700 0    50   ~ 0
+GPIO23
+Wire Wire Line
+	6400 3550 6400 3750
+Wire Wire Line
+	6400 3450 6500 3450
+Text Label 7100 3350 0    50   ~ 0
+GPIO23
 $EndSCHEMATC

Commit message: anteultimos_cambios
Parts:
- removed P2: CONN_02X05, MacroLib:Pin_strip_02x05, symbol EESTN5:CONN_02X05
- added P2: CONN_02x6, MacroLib:Pin_strip_2x6, symbol MacroLib:CONN_02x6
Connections:
- net BO1 is gone; now on net AO1: U1.4 (GPIO36)
- net BO2 is gone; now on net AIN2: U1.33 (GPIO21)
- net GPIO23 is gone; now on net AO2: U1.37 (GPIO23)
- net +5VF: now also P2.12
- net AIN1: now also U1.36 (GPIO22); no longer U1.31 (GPIO19)
- net AIN2: no longer U1.30 (GPIO18)
- net AO1: no longer U1.5 (GPIO39)
- net AO2: no longer U1.36 (GPIO22)
- net F+3.3V: now also P2.10
- net GND: now also P2.11
- net GPIO0: now also P2.2
- net GPIO25: now also P2.1
- net GPIO26: now also P2.3
- net GPIO32: now also P2.5
- net GPIO34: now also P2.9
- net GPIO35: now also P2.7
- net GPIO5: now also P2.4
- new net GPIO18: P2.6, U1.30 (GPIO18)
- new net GPIO19: P2.8, U1.31 (GPIO19)
- new net GPIO39: U1.5 (GPIO39)
Changed lines of the file:
@@
 Wire Wire Line
 	3000 2700 3100 2700
-Text Label 4750 3900 0    50   ~ 0
+Text Label 4500 3900 0    50   ~ 0
 GPIO0
 Wire Wire Line
-	4750 3900 4400 3900
+	4500 3900 4400 3900
 Text Label 4500 4000 0    50   ~ 0
 RXD
@@
 Text Label 3000 4000 2    50   ~ 0
 CLK
-Text GLabel 4500 3300 2    50   Input ~ 0
+Text GLabel 4500 2800 2    50   Input ~ 0
 AIN1
-Text GLabel 4500 3400 2    50   Input ~ 0
+Text GLabel 4500 3100 2    50   Input ~ 0
 AIN2
 Text GLabel 3000 3300 0    50   Input ~ 0
@@
 BIN2
 Wire Wire Line
-	4400 3300 4500 3300
+	4400 3100 4500 3100
 Wire Wire Line
 	3000 3600 3100 3600
 Wire Wire Line
-	4500 3400 4400 3400
-Wire Wire Line
-	4750 3500 4400 3500
-Text GLabel 3000 2900 0    50   Input ~ 0
+	4500 3300 4400 3300
+Wire Wire Line
+	4500 3500 4400 3500
+Text GLabel 3000 2800 0    50   Input ~ 0
 AO1
-Text GLabel 3000 2800 0    50   Input ~ 0
-BO1
-Text GLabel 4500 2800 2    50   Input ~ 0
+Text GLabel 4500 2700 2    50   Input ~ 0
 AO2
-Text GLabel 4500 3100 2    50   Input ~ 0
-BO2
 Wire Wire Line
 	3000 2800 3100 2800
-Wire Wire Line
-	3000 2900 3100 2900
 Wire Wire Line
 	4500 4000 4400 4000
@@
 GPIO35
 Wire Wire Line
-	3000 3000 3100 3000
+	2650 3000 3100 3000
 Wire Wire Line
 	3100 3100 2650 3100
@@
 Text Label 2650 3200 2    50   ~ 0
 GPIO32
-Text Label 4750 3500 0    50   ~ 0
+Text Label 4500 3500 0    50   ~ 0
 GPIO5
 Text Label 2650 3400 2    50   ~ 0
@@
 Text Label 2650 3500 2    50   ~ 0
 GPIO26
-Text GLabel 7100 3550 2    50   Input ~ 0
+Text GLabel 7100 3650 2    50   Input ~ 0
 +5VF
 $Comp
@@
 	1    0    0    -1
 $EndComp
-Text Label 4750 3600 0    50   ~ 0
+Text Label 4500 3600 0    50   ~ 0
 SDA
-Text Label 4750 3700 0    50   ~ 0
+Text Label 4500 3700 0    50   ~ 0
 SCL
 Wire Wire Line
-	4500 3100 4400 3100
-Wire Wire Line
 	4500 2800 4400 2800
 Wire Wire Line
@@
 	2750 3700 3100 3700
 Wire Wire Line
-	4750 4100 4400 4100
-Wire Wire Line
-	4400 3700 4750 3700
-Wire Wire Line
-	4400 3600 4750 3600
+	4500 4100 4400 4100
+Wire Wire Line
+	4400 3700 4500 3700
+Wire Wire Line
+	4400 3600 4500 3600
 Text Label 9350 2900 0    50   ~ 0
 RXD
@@
 Text Label 6400 3250 2    50   ~ 0
 GPIO26
-$Comp
-L EESTN5:CONN_02X05 P2
-U 1 1 60E67E8A
-P 6750 3350
-F 0 "P2" H 6750 3765 50  0000 C CNN
-F 1 "CONN_02X05" H 6750 3674 50  0000 C CNN
-F 2 "MacroLib:Pin_strip_02x05" H 6750 2150 50  0001 C CNN
-F 3 "" H 6750 2150 50  0000 C CNN
-	1    6750 3350
-	1    0    0    -1
-$EndComp
 Wire Wire Line
 	6400 3150 6500 3150
@@
 	6400 3250 6500 3250
 Wire Wire Line
+	7100 3650 7000 3650
+Wire Wire Line
+	7100 3150 7000 3150
+Wire Wire Line
+	7100 3250 7000 3250
+Wire Wire Line
+	7100 3350 7000 3350
+Wire Wire Line
 	7100 3550 7000 3550
-Wire Wire Line
-	7100 3150 7000 3150
-Wire Wire Line
-	7100 3250 7000 3250
-Wire Wire Line
-	7100 3350 7000 3350
-$Comp
-L power:GND #PWR06
-U 1 1 60E92CD9
-P 6400 3750
-F 0 "#PWR06" H 6400 3500 50  0001 C CNN
-F 1 "GND" H 6405 3577 50  0000 C CNN
-F 2 "" H 6400 3750 50  0001 C CNN
-F 3 "" H 6400 3750 50  0001 C CNN
-	1    6400 3750
-	-1   0    0    -1
-$EndComp
-Wire Wire Line
-	6400 3550 6500 3550
-Wire Wire Line
-	7100 3450 7000 3450
 Text Label 2150 2600 2    50   ~ 0
 F+3.3V
 Wire Wire Line
 	2150 2600 2250 2600
-Text Label 7100 3450 0    50   ~ 0
+Text Label 7100 3550 0    50   ~ 0
 F+3.3V
 Wire Wire Line
@@
 Text Label 6400 3150 2    50   ~ 0
 GPIO25
-Text GLabel 3000 3000 0    50   Input ~ 0
-GPIO34
+Text GLabel 3000 2900 0    50   Input ~ 0
+GPIO39
 Wire Notes Line
 	8050 1800 8050 5000
@@
 Wire Wire Line
 	3250 5100 3250 5350
-Text Label 4750 4100 0    50   ~ 0
+Text Label 4500 4100 0    50   ~ 0
 CS
 $Comp
@@
 Wire Wire Line
 	4500 2700 4400 2700
-Text Label 4500 2700 0    50   ~ 0
-GPIO23
-Wire Wire Line
-	6400 3550 6400 3750
+Text Label 4500 3300 0    50   ~ 0
+GPIO19
 Wire Wire Line
 	6400 3450 6500 3450
+Text Label 4500 3400 0    50   ~ 0
+GPIO18
+Wire Wire Line
+	4500 3400 4400 3400
+Wire Wire Line
+	3000 2900 3100 2900
+Text Label 2650 3000 2    50   ~ 0
+GPIO34
+$Comp
+L MacroLib:CONN_02x6 P2
+U 1 1 61691005
+P 6750 3400
+F 0 "P2" H 6750 3875 50  0000 C CNN
+F 1 "CONN_02x6" H 6750 3784 50  0000 C CNN
+F 2 "MacroLib:Pin_strip_2x6" H 6750 3800 50  0001 C CNN
+F 3 "" H 6750 3800 50  0001 C CNN
+	1    6750 3400
+	1    0    0    -1
+$EndComp
+Wire Wire Line
+	6400 3650 6400 3850
+Wire Wire Line
+	6400 3650 6500 3650
+$Comp
+L power:GND #PWR06
+U 1 1 60E92CD9
+P 6400 3850
+F 0 "#PWR06" H 6400 3600 50  0001 C CNN
+F 1 "GND" H 6405 3677 50  0000 C CNN
+F 2 "" H 6400 3850 50  0001 C CNN
+F 3 "" H 6400 3850 50  0001 C CNN
+	1    6400 3850
+	-1   0    0    -1
+$EndComp
+Text Label 6400 3550 2    50   ~ 0
+GPIO34
+Wire Wire Line
+	6400 3550 6500 3550
 Text Label 7100 3350 0    50   ~ 0
-GPIO23
+GPIO18
+Text Label 7100 3450 0    50   ~ 0
+GPIO19
+Wire Wire Line
+	7100 3450 7000 3450
 $EndSCHEMATC

Commit message: ultimos cambios
Parts:
- U1: footprint MacroLib:NodeMCU-ESP32 -> IAuto:NodeMCU-ESP32
Changed lines of the file:
@@
 F 0 "U1" H 3750 3265 50  0000 C CNN
 F 1 "ESP32_NODEMCU" H 3750 3174 50  0000 C CNN
-F 2 "MacroLib:NodeMCU-ESP32" H 3750 3400 50  0001 C CNN
+F 2 "IAuto:NodeMCU-ESP32" H 3750 3400 50  0001 C CNN
 F 3 "" H 3750 3400 50  0001 C CNN
 	1    3750 2800
