File: hardware/Potencia .sch (KiCad schematic (older format))
At the start: 54 parts, among them J1 Barrel_Jack_Switch, J2 4R7uH, J3 4R7uH, J4 M1, J5 M2, Q1 SI4835DDY-T1-GE3, Q2 2N7002, Q3 2N7002, Q4 2N7002, Q5 2N7002, U2 MP1584, U3 MP1584, U4 DRV8833

Commit message: hardware
Connections:
- net +5V: now also J4.5 (Pin_5), J5.2 (Pin_2), R18.1, R19.1, R22.1, R23.1
- net A1: now also J4.4 (Pin_4); no longer J4.3 (Pin_3)
- net AOUT1: now also J5.6 (Pin_6); no longer F3.1
- net AOUT2: now also F4.1; no longer J4.6 (Pin_6)
- net B1: now also J4.3 (Pin_3); no longer J4.4 (Pin_4)
- net BOUT1: now also J4.1 (Pin_1); no longer F4.1
- net BOUT2: now also F3.1; no longer J5.6 (Pin_6)
- net GND: now also J4.2 (Pin_2); no longer J4.5 (Pin_5)
- net at F3.2: now also J4.6 (Pin_6); no longer J4.1 (Pin_1)
- removed net +5C: J4.2 (Pin_2), J5.2 (Pin_2), R18.1, R19.1, R22.1, R23.1
- net GPIO35 renamed GPIO34
Changed lines of the file:
@@
 L EESTN5:Conn_01x06 J4
 U 1 1 60E9A461
-P 9300 2250
-F 0 "J4" H 9350 2550 50  0000 R CNN
-F 1 "M1" H 9350 1800 50  0000 R CNN
-F 2 "MacroLib:JST_XH_1X6" H 9300 2250 50  0001 C CNN
-F 3 "~" H 9300 2250 50  0001 C CNN
-	1    9300 2250
-	1    0    0    -1
+P 9300 2350
+F 0 "J4" H 9350 2650 50  0000 R CNN
+F 1 "M1" H 9350 1900 50  0000 R CNN
+F 2 "MacroLib:JST_XH_1X6" H 9300 2350 50  0001 C CNN
+F 3 "~" H 9300 2350 50  0001 C CNN
+	1    9300 2350
+	1    0    0    1
 $EndComp
 $Comp
@@
 Wire Wire Line
 	8650 4600 8750 4600
+Text Label 10300 1250 2    50   ~ 0
+AOUT2
+Wire Wire Line
+	9000 2550 9100 2550
 Text Label 9000 2550 2    50   ~ 0
-AOUT2
-Wire Wire Line
-	9000 2550 9100 2550
-Text Label 10300 1250 2    50   ~ 0
 BOUT1
 Wire Wire Line
 	10300 2050 10400 2050
-Text Label 10300 2550 2    50   ~ 0
+Text Label 9000 1250 2    50   ~ 0
 BOUT2
 Wire Wire Line
@@
 F 3 "" H 9950 2600 50  0001 C CNN
 	1    9950 2600
-	1    0    0    -1
-$EndComp
-$Comp
-L power:+5C #PWR029
-U 1 1 60DB9A93
-P 9950 1900
-F 0 "#PWR029" H 9950 1750 50  0001 C CNN
-F 1 "+5C" H 9965 2073 50  0000 C CNN
-F 2 "" H 9950 1900 50  0001 C CNN
-F 3 "" H 9950 1900 50  0001 C CNN
-	1    9950 1900
 	1    0    0    -1
 $EndComp
@@
 	6700 2550 6700 2350
 $Comp
-L power:+5C #PWR021
-U 1 1 610BCF85
-P 6700 2350
-F 0 "#PWR021" H 6700 2200 50  0001 C CNN
-F 1 "+5C" H 6715 2523 50  0000 C CNN
-F 2 "" H 6700 2350 50  0001 C CNN
-F 3 "" H 6700 2350 50  0001 C CNN
-	1    6700 2350
-	1    0    0    -1
-$EndComp
-$Comp
 L power:+3.3V #PWR018
 U 1 1 610BDD9C
@@
 Wire Wire Line
 	6700 1500 6700 1300
-$Comp
-L power:+5C #PWR020
-U 1 1 610CF2DE
-P 6700 1300
-F 0 "#PWR020" H 6700 1150 50  0001 C CNN
-F 1 "+5C" H 6715 1473 50  0000 C CNN
-F 2 "" H 6700 1300 50  0001 C CNN
-F 3 "" H 6700 1300 50  0001 C CNN
-	1    6700 1300
-	1    0    0    -1
-$EndComp
-$Comp
-L power:+3.3V #PWR017
-U 1 1 610CF2E4
-P 6200 1300
-F 0 "#PWR017" H 6200 1150 50  0001 C CNN
-F 1 "+3.3V" H 6215 1473 50  0000 C CNN
-F 2 "" H 6200 1300 50  0001 C CNN
-F 3 "" H 6200 1300 50  0001 C CNN
-	1    6200 1300
-	1    0    0    -1
-$EndComp
 Wire Wire Line
 	6100 1850 6200 1850
@@
 	7750 2550 7750 2350
 $Comp
-L power:+5C #PWR025
-U 1 1 610D8AB3
-P 7750 2350
-F 0 "#PWR025" H 7750 2200 50  0001 C CNN
-F 1 "+5C" H 7765 2523 50  0000 C CNN
-F 2 "" H 7750 2350 50  0001 C CNN
-F 3 "" H 7750 2350 50  0001 C CNN
-	1    7750 2350
-	1    0    0    -1
-$EndComp
-$Comp
 L power:+3.3V #PWR023
 U 1 1 610D8AB9
@@
 	7500 1400 7500 1650
 Wire Wire Line
-	7250 1400 7250 1300
-Connection ~ 7250 1400
-Wire Wire Line
 	7750 1500 7750 1300
-$Comp
-L power:+5C #PWR024
-U 1 1 610E2CE6
-P 7750 1300
-F 0 "#PWR024" H 7750 1150 50  0001 C CNN
-F 1 "+5C" H 7765 1473 50  0000 C CNN
-F 2 "" H 7750 1300 50  0001 C CNN
-F 3 "" H 7750 1300 50  0001 C CNN
-	1    7750 1300
-	1    0    0    -1
-$EndComp
-$Comp
-L power:+3.3V #PWR022
-U 1 1 610E2CEC
-P 7250 1300
-F 0 "#PWR022" H 7250 1150 50  0001 C CNN
-F 1 "+3.3V" H 7265 1473 50  0000 C CNN
-F 2 "" H 7250 1300 50  0001 C CNN
-F 3 "" H 7250 1300 50  0001 C CNN
-	1    7250 1300
-	1    0    0    -1
-$EndComp
 Wire Wire Line
 	7150 1850 7250 1850
@@
 Text Label 10300 2250 2    50   ~ 0
 A2
-Text Label 9000 1250 2    50   ~ 0
+Text Label 10300 2550 2    50   ~ 0
 AOUT1
 Wire Wire Line
@@
 Wire Wire Line
 	8650 2150 8650 1900
-$Comp
-L power:+5C #PWR027
-U 1 1 60DBA2B5
-P 8650 1900
-F 0 "#PWR027" H 8650 1750 50  0001 C CNN
-F 1 "+5C" H 8665 2073 50  0000 C CNN
-F 2 "" H 8650 1900 50  0001 C CNN
-F 3 "" H 8650 1900 50  0001 C CNN
-	1    8650 1900
-	1    0    0    -1
-$EndComp
 Wire Wire Line
 	7200 5000 7200 4900
@@
 	2000 1750 2000 1850
 Text GLabel 2200 1750 2    50   Input ~ 0
-GPIO35
+GPIO34
 Wire Wire Line
 	2350 4850 3650 4850
@@
 	7200 4400 7400 4400
 Connection ~ 7400 4400
+$Comp
+L power:+3.3V #PWR022
+U 1 1 610E2CEC
+P 7250 1300
+F 0 "#PWR022" H 7250 1150 50  0001 C CNN
+F 1 "+3.3V" H 7265 1473 50  0000 C CNN
+F 2 "" H 7250 1300 50  0001 C CNN
+F 3 "" H 7250 1300 50  0001 C CNN
+	1    7250 1300
+	1    0    0    -1
+$EndComp
+Connection ~ 7250 1400
+Wire Wire Line
+	7250 1400 7250 1300
+$Comp
+L power:+3.3V #PWR017
+U 1 1 610CF2E4
+P 6200 1300
+F 0 "#PWR017" H 6200 1150 50  0001 C CNN
+F 1 "+3.3V" H 6215 1473 50  0000 C CNN
+F 2 "" H 6200 1300 50  0001 C CNN
+F 3 "" H 6200 1300 50  0001 C CNN
+	1    6200 1300
+	1    0    0    -1
+$EndComp
+$Comp
+L power:+5V #PWR0102
+U 1 1 614A9D0E
+P 8650 1900
+F 0 "#PWR0102" H 8650 1750 50  0001 C CNN
+F 1 "+5V" H 8665 2073 50  0000 C CNN
+F 2 "" H 8650 1900 50  0001 C CNN
+F 3 "" H 8650 1900 50  0001 C CNN
+	1    8650 1900
+	1    0    0    -1
+$EndComp
+$Comp
+L power:+5V #PWR0103
+U 1 1 614AA1D9
+P 9950 1900
+F 0 "#PWR0103" H 9950 1750 50  0001 C CNN
+F 1 "+5V" H 9965 2073 50  0000 C CNN
+F 2 "" H 9950 1900 50  0001 C CNN
+F 3 "" H 9950 1900 50  0001 C CNN
+	1    9950 1900
+	1    0    0    -1
+$EndComp
+$Comp
+L power:+5V #PWR0104
+U 1 1 615094AA
+P 6700 1300
+F 0 "#PWR0104" H 6700 1150 50  0001 C CNN
+F 1 "+5V" H 6715 1473 50  0000 C CNN
+F 2 "" H 6700 1300 50  0001 C CNN
+F 3 "" H 6700 1300 50  0001 C CNN
+	1    6700 1300
+	1    0    0    -1
+$EndComp
+$Comp
+L power:+5V #PWR0105
+U 1 1 61509C4C
+P 7750 1300
+F 0 "#PWR0105" H 7750 1150 50  0001 C CNN
+F 1 "+5V" H 7765 1473 50  0000 C CNN
+F 2 "" H 7750 1300 50  0001 C CNN
+F 3 "" H 7750 1300 50  0001 C CNN
+	1    7750 1300
+	1    0    0    -1
+$EndComp
+$Comp
+L power:+5V #PWR0106
+U 1 1 6150A3AC
+P 7750 2350
+F 0 "#PWR0106" H 7750 2200 50  0001 C CNN
+F 1 "+5V" H 7765 2523 50  0000 C CNN
+F 2 "" H 7750 2350 50  0001 C CNN
+F 3 "" H 7750 2350 50  0001 C CNN
+	1    7750 2350
+	1    0    0    -1
+$EndComp
+$Comp
+L power:+5V #PWR0107
+U 1 1 6150A9C1
+P 6700 2350
+F 0 "#PWR0107" H 6700 2200 50  0001 C CNN
+F 1 "+5V" H 6715 2523 50  0000 C CNN
+F 2 "" H 6700 2350 50  0001 C CNN
+F 3 "" H 6700 2350 50  0001 C CNN
+	1    6700 2350
+	1    0    0    -1
+$EndComp
 $EndSCHEMATC

Commit message: anteultimos_cambios
Parts:
- removed Q2, Q4: 2N7002, EESTN5:SOT23, symbol EESTN5:2N7002
- removed R16, R18, R20, R22: 10K, EESTN5:R_0805, symbol EESTN5:R
Connections:
- net B1 is gone; now on net +5V: J4.3 (Pin_3)
- net B2 is gone; now on net +5V: J5.4 (Pin_4)
- net +5V: no longer J4.5 (Pin_5), J5.2 (Pin_2)
- net A1: now also J4.1 (Pin_1); no longer J4.4 (Pin_4)
- net A2: now also J5.1 (Pin_1); no longer J5.3 (Pin_3)
- net AOUT1: now also J5.5 (Pin_5); no longer J5.6 (Pin_6)
- net BOUT1: now also J4.5 (Pin_5); no longer J4.1 (Pin_1)
- net GND: now also J4.4 (Pin_4), J5.3 (Pin_3); no longer J4.2 (Pin_2), J5.5 (Pin_5)
- net at F4.2: now also J5.6 (Pin_6); no longer J5.1 (Pin_1)
- net GPIO34 renamed GPIO39
Other:
- moved on the sheet: Q3, Q5, R17, R19, R21, R23

Commit message: ultimos cambios
Connections:
- net AOUT1: now also F4.1; no longer J5.5 (Pin_5)
- net AOUT2: now also J5.5 (Pin_5); no longer F4.1
Changed lines of the file:
@@
 Wire Wire Line
 	8650 4600 8750 4600
-Text Label 10300 1250 2    50   ~ 0
+Text Label 10300 2150 2    50   ~ 0
 AOUT2
 Wire Wire Line
@@
 Text Label 10300 2550 2    50   ~ 0
 A2
-Text Label 10300 2150 2    50   ~ 0
+Text Label 10300 1250 2    50   ~ 0
 AOUT1
 Wire Wire Line

Commit message: Final
Parts:
- J4, J5: footprint MacroLib:JST_XH_1X6 -> IAuto:Conector_jst_6_pins_2mm
Connections:
- net +5V: now also J4.4 (Pin_4), J5.3 (Pin_3); no longer J4.3 (Pin_3), J5.4 (Pin_4)
- net A1: now also J4.6 (Pin_6); no longer J4.1 (Pin_1)
- net A2: now also J5.6 (Pin_6); no longer J5.1 (Pin_1)
- net AOUT2: now also J5.2 (Pin_2); no longer J5.5 (Pin_5)
- net BOUT1: now also J4.2 (Pin_2); no longer J4.5 (Pin_5)
- net GND: now also J4.3 (Pin_3), J5.4 (Pin_4); no longer J4.4 (Pin_4), J5.3 (Pin_3)
- net at F3.2: now also J4.1 (Pin_1); no longer J4.6 (Pin_6)
- net at F4.2: now also J5.1 (Pin_1); no longer J5.6 (Pin_6)
Changed lines of the file:
@@
 L EESTN5:Conn_01x06 J4
 U 1 1 60E9A461
-P 9300 2350
-F 0 "J4" H 9350 2650 50  0000 R CNN
-F 1 "M1" H 9350 1900 50  0000 R CNN
-F 2 "MacroLib:JST_XH_1X6" H 9300 2350 50  0001 C CNN
-F 3 "~" H 9300 2350 50  0001 C CNN
-	1    9300 2350
-	1    0    0    1
+P 9300 2250
+F 0 "J4" H 9350 2550 50  0000 R CNN
+F 1 "M1" H 9350 1800 50  0000 R CNN
+F 2 "IAuto:Conector_jst_6_pins_2mm" H 9300 2250 50  0001 C CNN
+F 3 "~" H 9300 2250 50  0001 C CNN
+	1    9300 2250
+	1    0    0    -1
 $EndComp
 $Comp
 L EESTN5:Conn_01x06 J5
 U 1 1 60E9ACC8
-P 10600 2350
-F 0 "J5" H 10650 2650 50  0000 R CNN
-F 1 "M2" H 10650 1900 50  0000 R CNN
-F 2 "MacroLib:JST_XH_1X6" H 10600 2350 50  0001 C CNN
-F 3 "~" H 10600 2350 50  0001 C CNN
-	1    10600 2350
-	1    0    0    1
+P 10600 2250
+F 0 "J5" H 10650 2550 50  0000 R CNN
+F 1 "M2" H 10650 1800 50  0000 R CNN
+F 2 "IAuto:Conector_jst_6_pins_2mm" H 10600 2250 50  0001 C CNN
+F 3 "~" H 10600 2250 50  0001 C CNN
+	1    10600 2250
+	1    0    0    -1
 $EndComp
 $Comp

Commit message: hardware_v20
Parts:
- added C12: 1000uF/16V, EESTN5:CAP_ELEC_8x11.5mm, symbol EESTN5:C
- added R16: 47k, EESTN5:R_0805, symbol EESTN5:R
- U4: footprint MacroLib:HTSSOP -> MacroLib:HTSSOPP
Connections:
- net +5V: now also C12.1
- net GND: now also U4.17 (GND_ppad), C12.2
- net VM: now also R16.1; no longer U4.1 (nSLEEP)
- new net: R16.2, U4.1 (nSLEEP)
Other:
- moved on the sheet: C1, C3, C5, C7, C9, D1, F2, J2, R11, R13, R3, R4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
